Commit message: Improved pnp and added MMAP learned policy

File: urdf/conveyor_g_path.urdf.xacro (robot description, xacro)
@@ -136,45 +136,45 @@
     </link>
     <joint name="joint_belt" type="fixed">
-      <origin xyz="0 0.3048 -0.105" rpy="0 0 0"/>
+      <origin xyz="0 0.3048 1.126" rpy="0 0 0"/>
       <parent link="world"/>
       <child link="link_belt"/>
     </joint>
     <joint name="joint_bridge_left" type="fixed">
-      <origin xyz="0.59689 0.3048 0.08415" rpy="0 0 0"/>
+      <origin xyz="0.59689 0.3048 1.23014" rpy="0 0 0"/>
       <parent link="world"/>
       <child link="link_bridge_left"/>
     </joint>
     <joint name="joint_bridge_right" type="fixed">
-      <origin xyz="-0.85089 0.3048 0.08415" rpy="0 0 0"/>
+      <origin xyz="-0.85089 0.3048 1.23014" rpy="0 0 0"/>
       <parent link="world"/>
       <child link="link_bridge_right"/>
     </joint>
     <joint name="joint_flap_back" type="fixed">
-      <origin xyz="0 0.0127 -0.0365" rpy="0 0 0"/>
+      <origin xyz="0 0.0127 1.182" rpy="0 0 0"/>
       <parent link="world"/>
       <child link="link_flap_back"/>
     </joint>
     <joint name="joint_flap_front" type="fixed">
-      <origin xyz="0 0.59689 -0.0365" rpy="0 0 0"/>
+      <origin xyz="0 0.59689 1.182" rpy="0 0 0"/>
       <parent link="world"/>
       <child link="link_flap_front"/>
     </joint>
     <joint name="joint_leg_back_left" type="fixed">
-      <origin xyz="0.68579 -0.0254 -0.54449" rpy="0 0 0"/>
+      <origin xyz="0.68579 -0.0254 0.556" rpy="0 0 0"/>
       <parent link="world"/>
       <child link="link_leg_back_left"/>
     </joint>
     <joint name="joint_leg_back_right" type="fixed">
-      <origin xyz="-0.68579 -0.0254 -0.54449" rpy="0 0 0"/>
+      <origin xyz="-0.68579 -0.0254 0.556" rpy="0 0 0"/>
       <parent link="world"/>
       <child link="link_leg_back_right"/>
     </joint>
     <joint name="joint_leg_front_left" type="fixed">
-      <origin xyz="0.68579 0.63499 -0.54449" rpy="0 0 0"/>
+      <origin xyz="0.68579 0.63499 0.556" rpy="0 0 0"/>
       <parent link="world"/>
       <child link="link_leg_front_left"/>
     </joint>
     <joint name="joint_leg_front_right" type="fixed">
-      <origin xyz="-0.68579 0.63499 -0.54449" rpy="0 0 0"/>
+      <origin xyz="-0.68579 0.63499 0.556" rpy="0 0 0"/>
       <parent link="world"/>
       <child link="link_leg_front_right"/>
