Commit message: Fixed conveyor

File: urdf/conveyor.urdf.xacro (robot description, xacro)
@@ -43,5 +43,5 @@
 	<origin rpy="0 0 0" xyz="0.75 -0.75 0" />
   	  <geometry>
-		<mesh filename="package://sawyer_irl_project/meshes/frame.stl"/>
+		<mesh filename="package://sawyer_irl_project/meshes/lab_conveyor/frame.stl"/>
 	  </geometry>
        </visual>
@@ -49,5 +49,5 @@
           <origin rpy="0 0 0" xyz="0.75 -0.75 0" />
   	  <geometry>
-		<mesh filename="package://sawyer_irl_project/meshes/conveyor_box.stl"/>
+		<mesh filename="package://sawyer_irl_project/meshes/lab_conveyor/conveyor_box.stl"/>
 	  </geometry>
 	</collision>
@@ -70,5 +70,5 @@
 	<origin rpy="0 0 0" xyz="0 0 0" />
   	  <geometry>
-		<mesh filename="package://sawyer_irl_project/meshes/belt.stl"/>
+		<mesh filename="package://sawyer_irl_project/meshes/lab_conveyor/belt.stl"/>
 	  </geometry>
        </visual>
@@ -76,5 +76,5 @@
           <origin rpy="0 0 0" xyz="0 0 0" />
   	  <geometry>
-		<mesh filename="package://sawyer_irl_project/meshes/belt.stl"/>
+		<mesh filename="package://sawyer_irl_project/meshes/lab_conveyor/belt.stl"/>
 	  </geometry>
 	</collision>
@@ -166,5 +166,5 @@
 	<origin rpy="0 0 0" xyz="0 0 0" />
   	  <geometry>
-		<mesh filename="package://sawyer_irl_project/meshes/roller.stl"/>
+		<mesh filename="package://sawyer_irl_project/meshes/lab_conveyor/roller.stl"/>
 	  </geometry>
        </visual>
@@ -195,5 +195,5 @@
 	<origin rpy="0 0 0" xyz="0 0 0" />
   	  <geometry>
-		<mesh filename="package://sawyer_irl_project/meshes/roller.stl"/>
+		<mesh filename="package://sawyer_irl_project/meshes/lab_conveyor/roller.stl"/>
 	  </geometry>
        </visual>
@@ -224,5 +224,5 @@
 	<origin rpy="0 0 0" xyz="0 0 0" />
   	  <geometry>
-		<mesh filename="package://sawyer_irl_project/meshes/roller.stl"/>
+		<mesh filename="package://sawyer_irl_project/meshes/lab_conveyor/roller.stl"/>
 	  </geometry>
        </visual>
@@ -253,5 +253,5 @@
 	    <origin rpy="0 0 0" xyz="0 0 0" />
   	  <geometry>
-		  <mesh filename="package://sawyer_irl_project/meshes/roller.stl"/>
+		  <mesh filename="package://sawyer_irl_project/meshes/lab_conveyor/roller.stl"/>
 	    </geometry>
       </visual>
@@ -282,5 +282,5 @@
 	<origin rpy="0 0 0" xyz="0 0 0" />
   	  <geometry>
-		<mesh filename="package://sawyer_irl_project/meshes/roller.stl"/>
+		<mesh filename="package://sawyer_irl_project/meshes/lab_conveyor/roller.stl"/>
 	  </geometry>
        </visual>
@@ -311,5 +311,5 @@
 	<origin rpy="0 0 0" xyz="0 0 0" />
   	  <geometry>
-		<mesh filename="package://sawyer_irl_project/meshes/roller.stl"/>
+		<mesh filename="package://sawyer_irl_project/meshes/lab_conveyor/roller.stl"/>
 	  </geometry>
        </visual>
@@ -340,5 +340,5 @@
 	<origin rpy="0 0 0" xyz="0 0 0" />
   	  <geometry>
-		<mesh filename="package://sawyer_irl_project/meshes/roller.stl"/>
+		<mesh filename="package://sawyer_irl_project/meshes/lab_conveyor/roller.stl"/>
 	  </geometry>
        </visual>
@@ -369,5 +369,5 @@
 	<origin rpy="0 0 0" xyz="0 0 0" />
   	  <geometry>
-		<mesh filename="package://sawyer_irl_project/meshes/roller.stl"/>
+		<mesh filename="package://sawyer_irl_project/meshes/lab_conveyor/roller.stl"/>
 	  </geometry>
        </visual>
@@ -398,5 +398,5 @@
 	<origin rpy="0 0 0" xyz="0 0 0" />
   	  <geometry>
-		<mesh filename="package://sawyer_irl_project/meshes/roller.stl"/>
+		<mesh filename="package://sawyer_irl_project/meshes/lab_conveyor/roller.stl"/>
 	  </geometry>
        </visual>
@@ -427,5 +427,5 @@
 	<origin rpy="0 0 0" xyz="0 0 0" />
   	  <geometry>
-		<mesh filename="package://sawyer_irl_project/meshes/roller.stl"/>
+		<mesh filename="package://sawyer_irl_project/meshes/lab_conveyor/roller.stl"/>
 	  </geometry>
        </visual>
@@ -456,5 +456,5 @@
 	<origin rpy="0 0 0" xyz="0 0 0" />
   	  <geometry>
-		<mesh filename="package://sawyer_irl_project/meshes/roller.stl"/>
+		<mesh filename="package://sawyer_irl_project/meshes/lab_conveyor/roller.stl"/>
 	  </geometry>
        </visual>
@@ -485,5 +485,5 @@
 	<origin rpy="0 0 0" xyz="0 0 0" />
   	  <geometry>
-		<mesh filename="package://sawyer_irl_project/meshes/roller.stl"/>
+		<mesh filename="package://sawyer_irl_project/meshes/lab_conveyor/roller.stl"/>
 	  </geometry>
        </visual>
@@ -514,5 +514,5 @@
 	<origin rpy="0 0 0" xyz="0 0 0" />
   	  <geometry>
-		<mesh filename="package://sawyer_irl_project/meshes/roller.stl"/>
+		<mesh filename="package://sawyer_irl_project/meshes/lab_conveyor/roller.stl"/>
 	  </geometry>
        </visual>
@@ -543,5 +543,5 @@
 	<origin rpy="0 0 0" xyz="0 0 0" />
   	  <geometry>
-		<mesh filename="package://sawyer_irl_project/meshes/roller.stl"/>
+		<mesh filename="package://sawyer_irl_project/meshes/lab_conveyor/roller.stl"/>
 	  </geometry>
        </visual>
@@ -572,5 +572,5 @@
 	<origin rpy="0 0 0" xyz="0 0 0" />
   	  <geometry>
-		<mesh filename="package://sawyer_irl_project/meshes/roller.stl"/>
+		<mesh filename="package://sawyer_irl_project/meshes/lab_conveyor/roller.stl"/>
 	  </geometry>
        </visual>
@@ -601,5 +601,5 @@
 	<origin rpy="0 0 0" xyz="0 0 0" />
   	  <geometry>
-		<mesh filename="package://sawyer_irl_project/meshes/roller.stl"/>
+		<mesh filename="package://sawyer_irl_project/meshes/lab_conveyor/roller.stl"/>
 	  </geometry>
        </visual>

File: urdf/conveyor_g_path.urdf.xacro (robot description, xacro)
@@ -11,5 +11,5 @@
         <origin xyz="0 0 0" rpy="0 0 0"/>
         <geometry>
-          <mesh filename="package://sawyer_irl_project/meshes/belt.dae" scale="0.001 0.001 0.001"/>
+          <mesh filename="package://sawyer_irl_project/meshes/vovrc_conveyor/belt.dae" scale="0.001 0.001 0.001"/>
         </geometry>
         <material name="191,191,191"/>
@@ -25,5 +25,5 @@
         <origin xyz="0 0 0" rpy="0 0 0"/>
         <geometry>
-          <mesh filename="package://sawyer_irl_project/meshes/bridge_left.dae" scale="0.001 0.001 0.001"/>
+          <mesh filename="package://sawyer_irl_project/meshes/vovrc_conveyor/bridge_left.dae" scale="0.001 0.001 0.001"/>
         </geometry>
         <material name="191,191,191"/>
@@ -39,5 +39,5 @@
         <origin xyz="0 0 0" rpy="0 0 0"/>
         <geometry>
-          <mesh filename="package://sawyer_irl_project/meshes/bridge_right.dae" scale="0.001 0.001 0.001"/>
+          <mesh filename="package://sawyer_irl_project/meshes/vovrc_conveyor/bridge_right.dae" scale="0.001 0.001 0.001"/>
         </geometry>
         <material name="191,191,191"/>
@@ -53,5 +53,5 @@
         <origin xyz="0 0 0" rpy="0 0 0"/>
         <geometry>
-          <mesh filename="package://sawyer_irl_project/meshes/flap_back.dae" scale="0.001 0.001 0.001"/>
+          <mesh filename="package://sawyer_irl_project/meshes/vovrc_conveyor/flap_back.dae" scale="0.001 0.001 0.001"/>
         </geometry>
         <material name="191,191,191"/>
@@ -67,5 +67,5 @@
         <origin xyz="0 0 0" rpy="0 0 0"/>
         <geometry>
-          <mesh filename="package://sawyer_irl_project/meshes/flap_front.dae" scale="0.001 0.001 0.001"/>
+          <mesh filename="package://sawyer_irl_project/meshes/vovrc_conveyor/flap_front.dae" scale="0.001 0.001 0.001"/>
         </geometry>
         <material name="191,191,191"/>
@@ -81,5 +81,5 @@
         <origin xyz="0 0 0" rpy="0 0 0"/>
         <geometry>
-          <mesh filename="package://sawyer_irl_project/meshes/leg_back_left.dae" scale="0.001 0.001 0.001"/>
+          <mesh filename="package://sawyer_irl_project/meshes/vovrc_conveyor/leg_back_left.dae" scale="0.001 0.001 0.001"/>
         </geometry>
         <material name="191,191,191"/>
@@ -95,5 +95,5 @@
         <origin xyz="0 0 0" rpy="0 0 0"/>
         <geometry>
-          <mesh filename="package://sawyer_irl_project/meshes/leg_back_right.dae" scale="0.001 0.001 0.001"/>
+          <mesh filename="package://sawyer_irl_project/meshes/vovrc_conveyor/leg_back_right.dae" scale="0.001 0.001 0.001"/>
         </geometry>
         <material name="191,191,191"/>
@@ -109,5 +109,5 @@
         <origin xyz="0 0 0" rpy="0 0 0"/>
         <geometry>
-          <mesh filename="package://sawyer_irl_project/meshes/leg_front_left.dae" scale="0.001 0.001 0.001"/>
+          <mesh filename="package://sawyer_irl_project/meshes/vovrc_conveyor/leg_front_left.dae" scale="0.001 0.001 0.001"/>
         </geometry>
         <material name="191,191,191"/>
@@ -123,5 +123,5 @@
         <origin xyz="0 0 0" rpy="0 0 0"/>
         <geometry>
-          <mesh filename="package://sawyer_irl_project/meshes/leg_front_right.dae" scale="0.001 0.001 0.001"/>
+          <mesh filename="package://sawyer_irl_project/meshes/vovrc_conveyor/leg_front_right.dae" scale="0.001 0.001 0.001"/>
         </geometry>
         <material name="191,191,191"/>
